File: attiny85_7seg.kicad_pcb (KiCad board)
At the start: 2 copper layers, 55 x 61 mm, 21 parts, among them J1 Conn_01x06_Pin, J2 Conn_01x03_Pin, U1 ATtiny85, U2 CC56-12SURKWA, U3 74HC595, U4 74HC595

Commit message: v0.0.5
Parts:
- added R5: 10k, Resistor_THT:R_Axial_DIN0207_L6.3mm_D2.5mm_P10.16mm_Horizontal, F.Cu at (151.3, 108.8)
- added SW1: SW_Push, Button_Switch_THT:SW_PUSH_6mm, F.Cu at (153.2, 98.0)
- moved J1 1.58 mm to (157.4, 90.3)
- moved J2 1.54 mm to (157.4, 85.4)
Routing:
- net /PB4: track 11.8 -> 30.2 mm
- net VCC: track 65.3 -> 81.8 mm, vias 0 -> 1
- net /PB0: track 38.5 -> 40.1 mm
- net /PB5: track 10.8 -> 12.4 mm
- net /PB3: track 60.9 -> 62.5 mm
- net /PB1: track 60.2 -> 61.8 mm
- net /PB2: track 59.8 -> 61.1 mm

Commit message: v0.0.6
Parts:
- added C1: 10uF, Capacitor_THT:C_Disc_D10.0mm_W2.5mm_P5.00mm, F.Cu at (109.4, 78.4)
- added C2: 10uF, Capacitor_THT:C_Disc_D10.0mm_W2.5mm_P5.00mm, F.Cu at (120.6, 78.4)
- added C3: 10uF, Capacitor_THT:C_Disc_D10.0mm_W2.5mm_P5.00mm, F.Cu at (120.1, 108.9)
