File: attiny85_7seg.kicad_sch (KiCad schematic)
At the start: 12 parts, among them J1 Conn_01x06_Pin, J2 Conn_01x03_Pin, U1 ATtiny85-20P, U2 CC56-12SURKWA, U3 74HC595, U4 74HC595

Commit message: 0.0.3
Parts:
- GND1, VCC1: footprint TestPoint:TestPoint_Pad_D1.5mm -> TestPoint:TestPoint_THTPad_3.0x3.0mm_Drill1.5mm
Other:
- title: v1.2.0 7seg display w/attiny85 & shift reg -> 7seg display w/attiny85 & shift reg
Changed lines of the file:
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@@
 	(paper "A4")
 	(title_block
-		(title "v1.2.0 7seg display w/attiny85 & shift reg")
-		(date "2026-06-06")
-		(rev "1.2.0")
-		(comment 4 "1.2.0: Fix pin headers footprint")
+		(title "7seg display w/attiny85 & shift reg")
+		(date "2026-06-09")
+		(rev "0.0.3")
+		(comment 4 "For changes check changes.md")
 	)
 	(junction
@@
 	)
 	(label "GND"
-		(at 105.41 38.1 180)
+		(at 105.41 38.1 270)
 		(effects
 			(font
@@
 			)
 		)
-		(property "Footprint" "TestPoint:TestPoint_Pad_D1.5mm"
+		(property "Footprint" "TestPoint:TestPoint_THTPad_3.0x3.0mm_Drill1.5mm"
 			(at 83.82 78.74 0)
 			(hide yes)
@@
 			)
 		)
-		(property "Footprint" "TestPoint:TestPoint_Pad_D1.5mm"
+		(property "Footprint" "TestPoint:TestPoint_THTPad_3.0x3.0mm_Drill1.5mm"
 			(at 83.82 116.84 0)
 			(hide yes)

Commit message: 0.0.4
Parts:
- U1: value ATtiny85-20P -> ATtiny85
Changed lines of the file:
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@@
 			)
 		)
-		(property "Value" "ATtiny85-20P"
+		(property "Value" "ATtiny85"
 			(at 69.85 93.9799 0)
 			(show_name no)

Commit message: v0.0.5
Parts:
- added R5: 10k, Resistor_THT:R_Axial_DIN0207_L6.3mm_D2.5mm_P10.16mm_Horizontal, symbol Device:R
- added SW1: SW_Push, Button_Switch_THT:SW_PUSH_6mm, symbol Switch:SW_Push
Connections:
- net GND: now also R5.2
- net PB4: now also R5.1, SW1.1
- net VCC: now also SW1.2

Commit message: v0.0.6
Parts:
- added C1, C2, C3: 10uF, Capacitor_THT:C_Disc_D10.0mm_W2.5mm_P5.00mm, symbol Device:C
Connections:
- net GND: now also C1.2, C2.2, C3.2
- net VCC: now also C1.1, C2.1, C3.1
