File: attiny85_7seg.kicad_sch (KiCad schematic)
At the start: 17 parts, among them J1 Conn_01x06_Pin, J2 Conn_01x03_Pin, SW1 SW_Push, U1 ATtiny85, U2 CC56-12SURKWA, U3 74HC595, U4 74HC595

Commit message: v0.1.0
Parts:
- removed GND1, VCC1: TestPoint, TestPoint:TestPoint_THTPad_3.0x3.0mm_Drill1.5mm, symbol Connector:TestPoint
- removed J1: Conn_01x06_Pin, Connector_PinHeader_2.54mm:PinHeader_1x06_P2.54mm_Vertical, symbol Connector:Conn_01x06_Pin
- removed J2: Conn_01x03_Pin, Connector_PinHeader_2.54mm:PinHeader_1x03_P2.54mm_Vertical, symbol Connector:Conn_01x03_Pin
- added C4: 10uF, Capacitor_THT:CP_Radial_D5.0mm_P2.50mm, symbol Device:C_Polarized
- added H1, H2, H3, H4: MountingHole, MountingHole:MountingHole_2.7mm_M2.5, symbol Mechanical:MountingHole
- added J2: Conn_01x02_Pin, Connector_Molex:Molex_KK-254_AE-6410-02A_1x02_P2.54mm_Vertical, symbol Connector:Conn_01x02_Pin
- added R6: 10k, Resistor_THT:R_Axial_DIN0207_L6.3mm_D2.5mm_P10.16mm_Horizontal, symbol Device:R
- added SW2: SW_Push, Button_Switch_THT:SW_PUSH_6mm, symbol Switch:SW_Push
- added TP1: TestPoint_2Pole, TestPoint:TestPoint_2Pads_Pitch2.54mm_Drill0.8mm, symbol Connector:TestPoint_2Pole
- C1, C2, C3: value 10uF -> 100nF
Connections:
- net PB5 is gone; now on net VCC: U1.1 (~{RESET}/PB5)
- net GND: now also C1.1, C4.1, J2.2 (Pin_2), R6.2, TP1.2; no longer C1.2
- net VCC: now also C1.2, C4.2, J2.1 (Pin_1), SW2.2, TP1.1; no longer C1.1
- net at R1.1: now also U2.12 (CC1); no longer U3.7 (QH)
- net D1: now reaches R1.2
- net D1: now also U3.7 (QH); no longer U2.12 (CC1)
- net at R4.1: now also U2.6 (CC4); no longer U4.2 (QC)
- net D4: now reaches R4.2
- net D4: now also U4.2 (QC); no longer U2.6 (CC4)
- net at R3.1: now also U2.8 (CC3); no longer U4.1 (QB)
- net at R2.1: now also U2.9 (CC2); no longer U4.15 (QA)
- net QE: now reaches U2.1 (e), U3.4 (QE)
- net QF: now reaches U2.10 (f), U3.5 (QF)
- net QA: now reaches U2.11 (a), U3.15 (QA)
- net QD: now reaches U2.2 (d), U3.3 (QD)
- net QC: now reaches U2.4 (c), U3.2 (QC)
- net QG: now reaches U2.5 (g), U3.6 (QG)
- net QB: now reaches U2.7 (b), U3.1 (QB)
- net D3: now reaches R3.2
- net D3: now also U4.1 (QB); no longer U2.8 (CC3)
- net D2: now reaches R2.2
- net D2: now also U4.15 (QA); no longer U2.9 (CC2)
- net PB0 renamed DATA
- net PB1 renamed SRCLK
- net PB2 renamed SRCLR
- net PB3 renamed RCLK
- net PB4 renamed MODE
- new net: R6.1, SW2.1
- no-connect marks 8 -> 7
Other:
- moved on the sheet: C1, C2, C3, R1, R2, R3, R4, U2

Commit message: v0.1.1
Parts:
- removed H1, H2, H3, H4: MountingHole, MountingHole:MountingHole_2.7mm_M2.5, symbol Mechanical:MountingHole
- added H1, H2, H3, H4: MountingHole_Pad, MountingHole:MountingHole_2.7mm_M2.5_DIN965_Pad_TopBottom, symbol Mechanical:MountingHole_Pad
Connections:
- net GND: now also H1.1, H2.1, H3.1, H4.1

Commit message: v0.1.2
Connections:
- net GND: now also C4.2; no longer C4.1
- net VCC: now also C4.1; no longer C4.2
Other:
- moved on the sheet: C4
Changed lines of the file:
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@@
 	(title_block
 		(title "7seg display w/attiny85 & shift reg")
-		(date "2026-07-28")
-		(rev "0.1.1")
+		(date "2026-08-18")
+		(rev "0.1.2")
 		(comment 4 "For changes check changes.md")
 	)
@@
 	(symbol
 		(lib_id "Device:C_Polarized")
-		(at 76.2 45.72 270)
+		(at 76.2 45.72 90)
 		(unit 1)
 		(body_style 1)
@@
 		(dnp no)
 		(property "Reference" "C4"
-			(at 75.438 38.1 90)
+			(at 76.962 53.34 90)
 			(show_name no)
 			(do_not_autoplace no)
@@
 		)
 		(property "Value" "10uF"
-			(at 75.438 40.64 90)
+			(at 76.962 50.8 90)
 			(show_name no)
 			(do_not_autoplace no)
@@
 		)
 		(property "Footprint" "Capacitor_THT:CP_Radial_D5.0mm_P2.50mm"
-			(at 72.39 46.6852 0)
+			(at 80.01 44.7548 0)
 			(hide yes)
 			(show_name no)
