File: kicad/attiny85_7seg.kicad_pcb (KiCad board)
At the start: 2 copper layers, 55 x 65 mm, 26 parts, among them J2 Conn_01x02_Pin, SW1 SW_Push, SW2 SW_Push, U1 ATtiny85, U2 CC56-12SURKWA, U3 74HC595, U4 74HC595

Commit message: v0.1.3
Connections:
- R6 pad 1: Net-(R6-Pad1) -> VCC
- R6 pad 2: GND -> Net-(R6-Pad2)
- SW2 pad 1: Net-(R6-Pad1) -> GND
- SW2 pad 2: VCC -> Net-(R6-Pad2)
Routing:
- net Net-(R6-Pad2): track 0.00 -> 32.8 mm
- net Net-(R6-Pad1): track 27.1 -> 0.00 mm
- net VCC: track 92.8 -> 97.2 mm
Changed lines of the file:
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@@
 	(title_block
 		(title "7seg display w/attiny85 & shift reg")
-		(date "2026-08-18")
-		(rev "0.1.2")
+		(date "2026-08-20")
+		(rev "0.1.3")
 		(comment 4 "For changes check changes.md")
 	)
@@
 			(layers "*.Cu" "*.Mask")
 			(remove_unused_layers no)
-			(net "Net-(R6-Pad1)")
+			(net "VCC")
 			(pintype "passive")
 		)
@@
 			(layers "*.Cu" "*.Mask")
 			(remove_unused_layers no)
-			(net "GND")
+			(net "Net-(R6-Pad2)")
 			(pintype "passive")
 		)
@@
 			(layers "*.Cu" "*.Mask")
 			(remove_unused_layers no)
-			(net "Net-(R6-Pad1)")
+			(net "GND")
 			(pinfunction "1_1")
 			(pintype "passive")
@@
 			(layers "*.Cu" "*.Mask")
 			(remove_unused_layers no)
-			(net "Net-(R6-Pad1)")
+			(net "GND")
 			(pinfunction "1_1")
 			(pintype "passive")
@@
 			(layers "*.Cu" "*.Mask")
 			(remove_unused_layers no)
-			(net "VCC")
+			(net "Net-(R6-Pad2)")
 			(pinfunction "2_2")
 			(pintype "passive")
@@
 			(layers "*.Cu" "*.Mask")
 			(remove_unused_layers no)
-			(net "VCC")
+			(net "Net-(R6-Pad2)")
 			(pinfunction "2_2")
 			(pintype "passive")
@@
 	)
 	(segment
-		(start 155.1861 117.6405)
-		(end 158.1211 117.6405)
-		(width 0.4)
-		(layer "F.Cu")
-		(net "VCC")
-	)
-	(segment
 		(start 158.2161 122.7005)
 		(end 158.8011 122.1155)
@@
 	)
 	(segment
+		(start 155.7356 118.19)
+		(end 158.6706 118.19)
+		(width 0.4)
+		(layer "F.Cu")
+		(net "VCC")
+	)
+	(segment
 		(start 169.0561 100.6305)
 		(end 168.1761 101.5105)
@@
 	)
 	(segment
-		(start 158.2161 129.2005)
-		(end 158.2161 122.7005)
+		(start 158.8011 118.3205)
+		(end 166.4211 118.3205)
 		(width 0.4)
 		(layer "F.Cu")
@@
 	)
 	(segment
-		(start 158.1211 117.6405)
+		(start 158.6706 118.19)
 		(end 158.8011 118.3205)
 		(width 0.4)
@@
 	)
 	(segment
+		(start 143.1561 129.2205)
+		(end 148.7961 129.2205)
+		(width 0.4)
+		(layer "F.Cu")
+		(net "VCC")
+	)
+	(segment
 		(start 148.8561 129.1605)
 		(end 148.8561 122.6605)
@@
 	)
 	(segment
-		(start 158.8011 122.1155)
-		(end 158.8011 118.3205)
+		(start 148.7961 129.2205)
+		(end 148.8561 129.1605)
 		(width 0.4)
 		(layer "F.Cu")
@@
 	)
 	(segment
+		(start 155.1861 117.6405)
+		(end 153.8761 117.6405)
+		(width 0.4)
+		(layer "F.Cu")
+		(net "VCC")
+	)
+	(segment
+		(start 143.2161 129.1605)
+		(end 143.1561 129.2205)
+		(width 0.4)
+		(layer "F.Cu")
+		(net "VCC")
+	)
+	(segment
+		(start 155.1861 117.6405)
+		(end 155.7356 118.19)
+		(width 0.4)
+		(layer "F.Cu")
+		(net "VCC")
+	)
+	(segment
 		(start 166.4211 118.3205)
 		(end 169.9211 121.8205)
@@
 	)
 	(segment
-		(start 162.7161 129.2005)
-		(end 162.7161 122.7005)
+		(start 149.1561 75.3605)
+		(end 158.1761 84.3805)
 		(width 0.2)
 		(layer "F.Cu")
-		(net "Net-(R6-Pad1)")
+		(net "Net-(U2-CC3)")
 	)
 	(segment
-		(start 144.3718 130.4362)
-		(end 143.1561 129.2205)
+		(start 158.1761 84.3805)
+		(end 158.1761 95.8005)
 		(width 0.2)
-		(layer "B.Cu")
-		(net "Net-(R6-Pad1)")
+		(layer "F.Cu")
+		(net "Net-(U2-CC3)")
 	)
 	(segment
-		(start 161.4804 130.4362)
-		(end 144.3718 130.4362)
+		(start 158.2161 129.2005)
+		(end 158.2161 123.1275)
 		(width 0.2)
-		(layer "B.Cu")
-		(net "Net-(R6-Pad1)")
+		(layer "F.Cu")
+		(net "Net-(R6-Pad2)")
 	)
 	(segment
-		(start 162.7161 129.2005)
-		(end 161.4804 130.4362)
+		(start 132.9961 129.2205)
+		(end 134.7956 131.02)
 		(width 0.2)
-		(layer "B.Cu")
-		(net "Net-(R6-Pad1)")
+		(layer "F.Cu")
+		(net "Net-(R6-Pad2)")
 	)
 	(segment
-		(start 149.1561 75.3605)
-		(end 158.1761 84.3805)
+		(start 134.7956 131.02)
+		(end 156.3966 131.02)
 		(width 0.2)
 		(layer "F.Cu")
-		(net "Net-(U2-CC3)")
+		(net "Net-(R6-Pad2)")
 	)
 	(segment
-		(start 158.1761 84.3805)
-		(end 158.1761 95.8005)
+		(start 156.3966 131.02)
+		(end 158.2161 129.2005)
 		(width 0.2)
 		(layer "F.Cu")
-		(net "Net-(U2-CC3)")
+		(net "Net-(R6-Pad2)")
 	)
 	(zone

Commit message: v0.1.31
Other:
- board text added: "M2.5"
Changed lines of the file:
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@@
 		(title "7seg display w/attiny85 & shift reg")
 		(date "2026-08-20")
-		(rev "0.1.3")
+		(rev "0.1.31")
 		(comment 4 "For changes check changes.md")
 	)
@@
 		)
 	)
+	(gr_text "M2.5"
+		(at 114 69.1 0)
+		(layer "User.1")
+		(effects
+			(font
+				(size 1 1)
+				(thickness 0.15)
+			)
+			(justify left bottom)
+		)
+	)
+	(dimension
+		(type orthogonal)
+		(layer "User.1")
+		(pts
+			(xy 121.204527 129.277073) (xy 121.204527 69.933927)
+		)
+		(height -5.534527)
+		(orientation 1)
+		(format
+			(prefix "")
+			(suffix "")
+			(units 3)
+			(units_format 0)
+			(precision 4)
+			(suppress_zeroes yes)
+		)
+		(style
+			(thickness 0.1)
+			(arrow_length 1.27)
+			(text_position_mode 0)
+			(arrow_direction outward)
+			(extension_height 0.58642)
+			(extension_offset 0.5)
+			(keep_text_aligned yes)
+		)
+		(gr_text "59.3431"
+			(at 114.52 99.6055 90)
+			(layer "User.1")
+			(effects
+				(font
+					(size 1 1)
+					(thickness 0.15)
+				)
+			)
+		)
+	)
+	(dimension
+		(type orthogonal)
+		(layer "User.1")
+		(pts
+			(xy 118.3761 67.1055) (xy 173.3761 67.1055)
+		)
+		(height -4.0855)
+		(orientation 0)
+		(format
+			(prefix "")
+			(suffix "")
+			(units 3)
+			(units_format 0)
+			(precision 4)
+			(suppress_zeroes yes)
+		)
+		(style
+			(thickness 0.1)
+			(arrow_length 1.27)
+			(text_position_mode 0)
+			(arrow_direction outward)
+			(extension_height 0.58642)
+			(extension_offset 0.5)
+			(keep_text_aligned yes)
+		)
+		(gr_text "55"
+			(at 145.8761 61.87 0)
+			(layer "User.1")
+			(effects
+				(font
+					(size 1 1)
+					(thickness 0.15)
+				)
+			)
+		)
+	)
+	(dimension
+		(type orthogonal)
+		(layer "User.1")
+		(pts
+			(xy 170.547673 69.933927) (xy 121.204527 69.933927)
+		)
+		(height -4.093927)
+		(orientation 0)
+		(format
+			(prefix "")
+			(suffix "")
+			(units 3)
+			(units_format 0)
+			(precision 4)
+			(suppress_zeroes yes)
+		)
+		(style
+			(thickness 0.1)
+			(arrow_length 1.27)
+			(text_position_mode 0)
+			(arrow_direction outward)
+			(extension_height 0.58642)
+			(extension_offset 0.5)
+			(keep_text_aligned yes)
+		)
+		(gr_text "49.3431"
+			(at 145.8761 64.69 0)
+			(layer "User.1")
+			(effects
+				(font
+					(size 1 1)
+					(thickness 0.15)
+				)
+			)
+		)
+	)
+	(dimension
+		(type orthogonal)
+		(layer "User.1")
+		(pts
+			(xy 118.3761 132.1055) (xy 118.3761 67.1055)
+		)
+		(height -6.2361)
+		(orientation 1)
+		(format
+			(prefix "")
+			(suffix "")
+			(units 3)
+			(units_format 0)
+			(precision 4)
+			(suppress_zeroes yes)
+		)
+		(style
+			(thickness 0.1)
+			(arrow_length 1.27)
+			(text_position_mode 0)
+			(arrow_direction outward)
+			(extension_height 0.58642)
+			(extension_offset 0.5)
+			(keep_text_aligned yes)
+		)
+		(gr_text "65"
+			(at 110.99 99.6055 90)
+			(layer "User.1")
+			(effects
+				(font
+					(size 1 1)
+					(thickness 0.15)
+				)
+			)
+		)
+	)
 	(segment
 		(start 158.2161 122.7005)
@@
 	)
 	(segment
-		(start 149.1561 75.3605)
-		(end 158.1761 84.3805)
-		(width 0.2)
-		(layer "F.Cu")
-		(net "Net-(U2-CC3)")
-	)
-	(segment
-		(start 158.1761 84.3805)
-		(end 158.1761 95.8005)
-		(width 0.2)
-		(layer "F.Cu")
-		(net "Net-(U2-CC3)")
-	)
-	(segment
 		(start 158.2161 129.2005)
 		(end 158.2161 123.1275)
@@
 		(net "Net-(R6-Pad2)")
 	)
+	(segment
+		(start 149.1561 75.3605)
+		(end 158.1761 84.3805)
+		(width 0.2)
+		(layer "F.Cu")
+		(net "Net-(U2-CC3)")
+	)
+	(segment
+		(start 158.1761 84.3805)
+		(end 158.1761 95.8005)
+		(width 0.2)
+		(layer "F.Cu")
+		(net "Net-(U2-CC3)")
+	)
 	(zone

Commit message: v0.1.32
Parts:
- added J1: Conn_01x06_Pin, Connector_PinHeader_2.54mm:PinHeader_2x03_P2.54mm_Vertical, F.Cu at (149.0, 110.2)
- moved C1 1.53 mm to (156.7, 112.6)
- moved U1 1.23 mm to (167.7, 118.3)
- moved J2 0.97 mm to (169.1, 99.7)
Connections:
- R6 pad 2: Net-(R6-Pad2) -> /RST
- SW2 pad 2: Net-(R6-Pad2) -> /RST
- U1 pad 1: VCC -> /RST
Routing:
- net /RST: track 0.00 -> 54.1 mm, vias 0 -> 1
- net Net-(R6-Pad2): track 32.8 -> 0.00 mm
- net /RCLK: track 59.2 -> 79.0 mm
- net /SRCLK: track 52.0 -> 64.4 mm
- net /MODE: track 34.8 -> 46.1 mm
- net /SRCLR: track 52.3 -> 63.6 mm, vias 0 -> 1
- net VCC: track 97.2 -> 90.5 mm
- net /DATA: track 39.4 -> 41.9 mm
- net /D3: track 21.8 -> 23.6 mm
- net /D4: track 19.7 -> 21.2 mm, vias 0 -> 1
Other:
- board text added: "0"
- board text added: "1"
- board text added: "5"
- board text removed: "Pin headers used only for programming Attiny85"

Commit message: v0.1.41
Parts:
- added C5: 100nF, Capacitor_THT:C_Disc_D10.0mm_W2.5mm_P5.00mm, F.Cu at (131.7, 129.2)
- added C6: 100nF, Capacitor_THT:C_Disc_D10.0mm_W2.5mm_P5.00mm, F.Cu at (126.7, 125.4)
- moved R5 8.34 mm to (135.7, 129.2), turned to 0 degrees
- moved R6 4.70 mm to (145.9, 125.4)
Routing:
- net /RCLK: track 79.0 -> 55.6 mm, vias 1 -> 0
- net /DATA: track 41.9 -> 26.8 mm, vias 0 -> 1
- net /MODE: track 46.1 -> 57.0 mm
- net /D4: track 21.2 -> 25.1 mm
- net /QG: track 32.4 -> 29.2 mm
- net VCC: track 90.5 -> 87.3 mm
- net /SRCLK: track 64.4 -> 63.0 mm
- net Net-(U2-CC1): track 24.5 -> 25.6 mm
- net /RST: track 54.1 -> 54.8 mm
- net /D3: track 23.6 -> 23.0 mm
- net /D2: track 32.6 -> 33.1 mm
