File: kicad/attiny85_7seg.kicad_sch (KiCad schematic)
At the start: 22 parts, among them J2 Conn_01x02_Pin, SW1 SW_Push, SW2 SW_Push, U1 ATtiny85, U2 CC56-12SURKWA, U3 74HC595, U4 74HC595

Commit message: v0.1.3
Connections:
- net GND: now also SW2.1; no longer R6.2
- net VCC: now also R6.1; no longer SW2.2
- new net: R6.2, SW2.2
Other:
- moved on the sheet: R6, SW2
Changed lines of the file:
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@@
 	(title_block
 		(title "7seg display w/attiny85 & shift reg")
-		(date "2026-08-18")
-		(rev "0.1.2")
+		(date "2026-08-20")
+		(rev "0.1.3")
 		(comment 4 "For changes check changes.md")
 	)
@@
 	)
 	(junction
-		(at 73.66 135.89)
+		(at 73.66 134.62)
 		(diameter 0)
 		(color 0 0 0 0)
@@
 	(wire
 		(pts
-			(xy 67.31 135.89) (xy 73.66 135.89)
-		)
-		(stroke
-			(width 0)
-			(type default)
-		)
-	)
-	(wire
-		(pts
 			(xy 92.71 157.48) (xy 92.71 162.56)
 		)
@@
 	(wire
 		(pts
-			(xy 142.24 100.33) (xy 142.24 106.68)
+			(xy 73.66 154.94) (xy 73.66 162.56)
 		)
 		(stroke
@@
 	(wire
 		(pts
-			(xy 73.66 157.48) (xy 73.66 162.56)
+			(xy 142.24 100.33) (xy 142.24 106.68)
 		)
 		(stroke
@@
 	(wire
 		(pts
+			(xy 67.31 134.62) (xy 73.66 134.62)
+		)
+		(stroke
+			(width 0)
+			(type default)
+		)
+	)
+	(wire
+		(pts
 			(xy 83.82 67.31) (xy 83.82 76.2)
 		)
@@
 	(wire
 		(pts
+			(xy 73.66 134.62) (xy 73.66 135.89)
+		)
+		(stroke
+			(width 0)
+			(type default)
+		)
+	)
+	(wire
+		(pts
 			(xy 168.91 115.57) (xy 168.91 118.11)
 		)
@@
 	(wire
 		(pts
-			(xy 73.66 130.81) (xy 73.66 135.89)
+			(xy 73.66 130.81) (xy 73.66 134.62)
 		)
 		(stroke
@@
 	(wire
 		(pts
-			(xy 152.4 71.12) (xy 160.02 71.12)
+			(xy 73.66 143.51) (xy 73.66 144.78)
 		)
 		(stroke
@@
 	(wire
 		(pts
-			(xy 251.46 97.79) (xy 251.46 104.14)
+			(xy 152.4 71.12) (xy 160.02 71.12)
 		)
 		(stroke
@@
 	(wire
 		(pts
-			(xy 152.4 78.74) (xy 152.4 96.52)
+			(xy 251.46 97.79) (xy 251.46 104.14)
 		)
 		(stroke
@@
 	(wire
 		(pts
-			(xy 264.16 104.14) (xy 271.78 104.14)
+			(xy 152.4 78.74) (xy 152.4 96.52)
 		)
 		(stroke
@@
 	(wire
 		(pts
-			(xy 73.66 135.89) (xy 73.66 139.7)
+			(xy 264.16 104.14) (xy 271.78 104.14)
 		)
 		(stroke
@@
 	)
 	(label "RESET"
-		(at 67.31 135.89 0)
+		(at 67.31 134.62 0)
 		(effects
 			(font
@@
 	(symbol
 		(lib_id "Switch:SW_Push")
-		(at 73.66 144.78 90)
+		(at 73.66 149.86 90)
 		(unit 1)
 		(body_style 1)
@@
 		(fields_autoplaced yes)
 		(property "Reference" "SW2"
-			(at 74.93 143.5099 90)
+			(at 74.93 148.5899 90)
 			(show_name no)
 			(do_not_autoplace no)
@@
 		)
 		(property "Value" "SW_Push"
-			(at 74.93 146.0499 90)
+			(at 74.93 151.1299 90)
 			(show_name no)
 			(do_not_autoplace no)
@@
 		)
 		(property "Footprint" "Button_Switch_THT:SW_PUSH_6mm"
-			(at 68.58 144.78 0)
+			(at 68.58 149.86 0)
 			(hide yes)
 			(show_name no)
@@
 		)
 		(property "Datasheet" ""
-			(at 68.58 144.78 0)
+			(at 68.58 149.86 0)
 			(hide yes)
 			(show_name no)
@@
 		)
 		(property "Description" "Push button switch, generic, two pins"
-			(at 73.66 144.78 0)
+			(at 73.66 149.86 0)
 			(hide yes)
 			(show_name no)
@@
 	(symbol
 		(lib_id "Device:R")
-		(at 73.66 153.67 0)
+		(at 73.66 139.7 0)
 		(unit 1)
 		(body_style 1)
@@
 		(fields_autoplaced yes)
 		(property "Reference" "R6"
-			(at 76.2 152.3999 0)
+			(at 76.2 138.4299 0)
 			(show_name no)
 			(do_not_autoplace no)
@@
 		)
 		(property "Value" "10k"
-			(at 76.2 154.9399 0)
+			(at 76.2 140.9699 0)
 			(show_name no)
 			(do_not_autoplace no)
@@
 		)
 		(property "Footprint" "Resistor_THT:R_Axial_DIN0207_L6.3mm_D2.5mm_P10.16mm_Horizontal"
-			(at 71.882 153.67 90)
+			(at 71.882 139.7 90)
 			(hide yes)
 			(show_name no)
@@
 		)
 		(property "Datasheet" ""
-			(at 73.66 153.67 0)
+			(at 73.66 139.7 0)
 			(hide yes)
 			(show_name no)
@@
 		)
 		(property "Description" "Resistor"
-			(at 73.66 153.67 0)
+			(at 73.66 139.7 0)
 			(hide yes)
 			(show_name no)

Commit message: v0.1.32
Parts:
- added J1: Conn_01x06_Pin, Connector_PinHeader_2.54mm:PinHeader_2x03_P2.54mm_Vertical, symbol Connector:Conn_01x06_Pin
Connections:
- net DATA: now also J1.1 (Pin_1)
- net MODE: now also J1.5 (Pin_5)
- net RCLK: now also J1.4 (Pin_4)
- net SRCLK: now also J1.2 (Pin_2)
- net SRCLR: now also J1.3 (Pin_3)
- net VCC: no longer U1.1 (~{RESET}/PB5)
- net RST: now reaches R6.2, SW2.2
- net RST: now also U1.1 (~{RESET}/PB5), J1.6 (Pin_6)
Other:
- note added: "Fix pull donw and pull up button"

Commit message: v0.1.41
Parts:
- added C5, C6: 100nF, Capacitor_THT:C_Disc_D10.0mm_W2.5mm_P5.00mm, symbol Device:C
Connections:
- net GND: now also C5.2, C6.1
- net MODE: now also C5.1
- net RST: now also C6.2
Other:
- moved on the sheet: SW2

Commit message: v0.1.42
Parts:
- removed C6: 100nF, Capacitor_THT:C_Disc_D10.0mm_W2.5mm_P5.00mm, symbol Device:C
Connections:
- net MODE: now also U1.7 (PB2); no longer U1.3 (XTAL2/PB4)
- net SRCLR: now also U1.3 (XTAL2/PB4); no longer U1.7 (PB2)
Other:
- note added: "Add sw debounce to MODE"
- note removed: "Fix pull donw and pull up button"
- moved on the sheet: R5, R6, SW1, SW2

Commit message: v0.1.50
Parts:
- added C6: 100nF, Capacitor_THT:C_Disc_D10.0mm_W2.5mm_P5.00mm, symbol Device:C
Connections:
- net GND: now also C6.2
- net RST: now also C6.1
Other:
- note added: "C5 & C6 are in case of signal degredation"
- moved on the sheet: R6, SW2
